File: KiCad/3dFilamentDryer/3dFilamentDryer.kicad_pcb (KiCad board)
At the start: 2 copper layers, 162.5 x 47 mm, 47 parts, among them J1 ILI9341 Connection Port, J2 FTDI, J3 Mains, J4 Fan, J5 MAX6675, Q1 BTA12-600BW, Q2 S8050-J3Y, Q3 S8050-J3Y, U1 4N28, U2 TLV1117-33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

Commit message: v1.2
Parts:
- added D5: MMSD4148T1G, Diode_SMD:D_SOD-123, F.Cu at (138.0, 109.5)
- added K1: SRD-05VDC-SL-C, Relay_THT:Relay_SPDT_SANYOU_SRD_Series_Form_C, F.Cu at (125.0, 109.5)
- added Q4: BC817-25-HT, Package_TO_SOT_SMD:SOT-23, F.Cu at (129.1, 107.5)
- added R15: 10k, Resistor_SMD:R_0402_1005Metric, F.Cu at (137.0, 106.0)
- added R16: 1k, Resistor_SMD:R_0402_1005Metric, F.Cu at (132.5, 108.0)
- U3: value ESP32-WROOM-32 -> ESP32-WROOM-32E-N4; footprint RF_Module:ESP32-WROOM-32 -> RF_Module:ESP32-WROOM-32E
- moved RV1 4.50 mm to (100.2, 85.2)
- moved U3 3.04 mm to (202.5, 87.8)
- moved C1 2.75 mm to (108.0, 83.5)
- moved L1 2.75 mm to (119.0, 91.0)
- moved RV2 2.26 mm to (132.8, 112.8)
Connections:
- J4 pad 1: LINE -> Net-(J4-Pin_1)
- U3 pad 14: unconnected-(U3-IO12-Pad14) -> /FAN
Routing:
- net +5V: track 85.4 -> 154.0 mm
- net /FAN: track 0.00 -> 65.7 mm, vias 0 -> 4
- net Net-(J4-Pin_1): track 0.00 -> 49.0 mm
- net LINE: track 54.6 -> 94.2 mm
- net GND: track 0.00 -> 23.3 mm, vias 0 -> 4
- net Net-(D5-A): track 0.00 -> 20.8 mm
- net Net-(Q1-A2): track 77.2 -> 59.3 mm
- net Net-(Q4-B): track 0.00 -> 8.42 mm
- net Net-(C1-Pad2): track 31.1 -> 34.0 mm
- net Net-(PS1-AC/L): track 50.8 -> 52.0 mm
- net Net-(Q1-A1): track 52.7 -> 51.8 mm
- net Net-(C1-Pad1): track 30.7 -> 30.2 mm
