File: KiCad/3dFilamentDryer/3dFilamentDryer.kicad_pcb (KiCad board)
At the start: 2 copper layers, 162.5 x 47 mm, 52 parts, among them J1 ILI9341 Connection Port, J2 FTDI, J3 Mains, J4 Fan, J5 MAX6675, K1 SRD-05VDC-SL-C, Q1 BTA12-600BW, Q2 S8050-J3Y, Q3 S8050-J3Y, Q4 BC817-25-HT, U1 4N28, U2 TLV1117-33, U3 ESP32-WROOM-32E-N4, U5 MOC3053M, U6 SN74LVC1G14DBVR

Commit message: Rev 1.2 KiCad design update with fan/relay control, BOM and gerber outputs
Co-Authored-By: Claude Opus 4.6 (1M context) <noreply@anthropic.com>
Routing:
- net GND: vias 4 -> 86
