File: KiCad/3dFilamentDryer/3dFilamentDryer.kicad_pcb (KiCad board)
At the start: 2 copper layers, 162.5 x 47 mm, 52 parts, among them J1 ILI9341 Connection Port, J2 FTDI, J3 Mains, J4 Fan, J5 MAX6675, K1 SRD-05VDC-SL-C, Q1 BTA12-600BW, Q2 S8050-J3Y, Q3 S8050-J3Y, Q4 BC817-25-HT, U1 4N28, U2 TLV1117-33, U3 ESP32-WROOM-32E-N4, U5 MOC3053M, U6 SN74LVC1G14DBVR

Commit message: PCB fix
Connections:
- J1 pad 10: Net-(J1-SCK) -> /VSPI_SCK
- J1 pad 12: Net-(J1-SDI(MOSI)) -> /VSPI_MOSI
- J1 pad 13: Net-(J1-SDO(MISO)) -> /VSPI_MISO
- J1 pad 6: Net-(J1-SDI(MOSI)) -> /VSPI_MOSI
- J1 pad 7: Net-(J1-SCK) -> /VSPI_SCK
- J1 pad 9: Net-(J1-SDO(MISO)) -> /VSPI_MISO
- J5 pad 3: Net-(J1-SCK) -> /VSPI_SCK
- J5 pad 4: Net-(J5-Pin_4) -> /SENSOR_CS
- J5 pad 5: Net-(J1-SDO(MISO)) -> /VSPI_MISO
- U3 pad 11: unconnected-(U3-IO26-Pad11) -> /SENSOR_CS
- U3 pad 13: unconnected-(U3-IO14-Pad13) -> Net-(J1-RESET)
- U3 pad 14: /FAN -> unconnected-(U3-IO12-Pad14)
- U3 pad 16: Net-(J5-Pin_4) -> /FAN
- U3 pad 20: Net-(J1-SCK) -> unconnected-(U3-SCK/CLK-Pad20)
- U3 pad 21: Net-(J1-SDI(MOSI)) -> unconnected-(U3-SDO/SD0-Pad21)
- U3 pad 22: Net-(J1-SDO(MISO)) -> unconnected-(U3-SDI/SD1-Pad22)
- U3 pad 23: Net-(J1-CS) -> unconnected-(U3-IO15-Pad23)
- U3 pad 24: Net-(J1-DC) -> unconnected-(U3-IO2-Pad24)
- U3 pad 26: Net-(J1-RESET) -> Net-(J1-CS)
- U3 pad 27: unconnected-(U3-IO16-Pad27) -> Net-(J1-DC)
- U3 pad 30: unconnected-(U3-IO18-Pad30) -> /VSPI_SCK
- U3 pad 31: unconnected-(U3-IO19-Pad31) -> /VSPI_MISO
- U3 pad 37: unconnected-(U3-IO23-Pad37) -> /VSPI_MOSI
Routing:
- net Net-(J1-SDO(MISO)): track 61.4 -> 0.00 mm, vias 1 -> 0
- net /VSPI_SCK: track 0.00 -> 55.4 mm, vias 0 -> 2
- net /VSPI_MISO: track 0.00 -> 53.7 mm, vias 0 -> 3
- net Net-(J1-SCK): track 51.2 -> 0.00 mm, vias 3 -> 0
- net Net-(J1-SDI(MOSI)): track 51.0 -> 0.00 mm, vias 1 -> 0
- net /SENSOR_CS: track 0.00 -> 43.5 mm, vias 0 -> 2
- net /VSPI_MOSI: track 0.00 -> 29.8 mm
- net Net-(J5-Pin_4): track 29.1 -> 0.00 mm, vias 2 -> 0
- net Net-(Q1-A2): track 59.3 -> 75.7 mm
- net Net-(J1-RESET): track 19.5 -> 35.7 mm, vias 0 -> 1
- net /FAN: track 65.7 -> 70.4 mm
- net Net-(J1-DC): track 23.8 -> 19.8 mm, vias 0 -> 3
- net Net-(J1-CS): track 21.2 -> 22.1 mm
- net +3V3: track 114.2 -> 113.6 mm
- net GND: vias 86 -> 127

Commit message: Firmware v2.1.2 Hardware Rev2
Parts:
- removed F2: 250VAC 1A Slow Blow, Fuse:Fuseholder_Clip-5x20mm_Littelfuse_445-030_Inline_P20.50x5.20mm_D1.30mm_Horizontal
- removed F4: 250VAC 2.5A Normal, Fuse:Fuseholder_Clip-5x20mm_Littelfuse_445-030_Inline_P20.50x5.20mm_D1.30mm_Horizontal
- F3: value 250VAC 2.5A Normal -> 250VAC 8A Normal
- R1: value Heater 500W -> Heater 1300W
Connections:
- C1 pad 2: Net-(C1-Pad2) -> NEUT
- L1 pad 1: Net-(C1-Pad2) -> NEUT
- R1 pad 2: Net-(F4-Pad2) -> NEUT
- RV1 pad 2: Net-(C1-Pad2) -> NEUT
Routing:
- net NEUT: track 53.4 -> 124.1 mm, vias 0 -> 5
- net Net-(C1-Pad2): track 34.0 -> 0.00 mm
- net Net-(F4-Pad2): track 12.1 -> 0.00 mm
- net GND: vias 127 -> 170
