File: KiCad/3dFilamentDryer/3dFilamentDryer.kicad_sch (KiCad schematic)
At the start: 47 parts, among them J1 ILI9341 Connection Port, J2 FTDI, J3 Mains, J4 Fan, J5 MAX6675, Q1 BTA12-600BW, Q2 S8050-J3Y, Q3 S8050-J3Y, U1 4N28, U2 TLV1117-33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

Commit message: v1.2
Parts:
- added D5: MMSD4148T1G, Diode_SMD:D_SOD-123, symbol Diode:MMSD4148
- added K1: SRD-05VDC-SL-C, Relay_THT:Relay_SPDT_SANYOU_SRD_Series_Form_C, symbol Relay:SANYOU_SRD_Form_C
- added Q4: BC817-25-HT, Package_TO_SOT_SMD:SOT-23, symbol Transistor_BJT:BC817
- added R15: 10k, Resistor_SMD:R_0402_1005Metric, symbol Device:R
- added R16: 1k, Resistor_SMD:R_0402_1005Metric, symbol Device:R
- U3: value ESP32-WROOM-32 -> ESP32-WROOM-32E-N4; footprint RF_Module:ESP32-WROOM-32 -> RF_Module:ESP32-WROOM-32E
Connections:
- net +5V: now also D5.1 (K), K1.2
- net GND: now also Q4.2 (E), R15.2
- net LINE: now also K1.1; no longer J4.1 (Pin_1)
- net FAN: now reaches U3.14 (IO12)
- net FAN: now also R16.2
- new net: J4.1 (Pin_1), K1.3
- new net: D5.2 (A), K1.5, Q4.3 (C)
- new net: Q4.1 (B), R15.1, R16.1
Other:
- note added: "Fan Control"
- note removed: "Mains Terminals"
- moved on the sheet: J3, J4
