File: KiCad/3dFilamentDryer/3dFilamentDryer.kicad_sch (KiCad schematic)
At the start: 52 parts, among them J1 ILI9341 Connection Port, J2 FTDI, J3 Mains, J4 Fan, J5 MAX6675, K1 SRD-05VDC-SL-C, Q1 BTA12-600BW, Q2 S8050-J3Y, Q3 S8050-J3Y, Q4 BC817-25-HT, U1 4N28, U2 TLV1117-33, U3 ESP32-WROOM-32E-N4, U5 MOC3053M, U6 SN74LVC1G14DBVR

Commit message: Rev 1.2 KiCad design update with fan/relay control, BOM and gerber outputs
Co-Authored-By: Claude Opus 4.6 (1M context) <noreply@anthropic.com>
Parts:
- added V1: VSIN, symbol Simulation_SPICE:VSIN
Connections:
- net LINE: now also V1.1
- net NEUT: now also V1.2
Changed lines of the file:
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@@
 	)
 	(junction
+		(at 377.19 167.64)
+		(diameter 0)
+		(color 0 0 0 0)
+	)
+	(junction
 		(at 130.81 91.44)
 		(diameter 0)
@@
 	)
 	(junction
+		(at 377.19 177.8)
+		(diameter 0)
+		(color 0 0 0 0)
+	)
+	(junction
 		(at 337.82 80.01)
 		(diameter 0)
@@
 	(wire
 		(pts
-			(xy 377.19 173.99) (xy 377.19 179.07)
+			(xy 377.19 173.99) (xy 377.19 177.8)
 		)
 		(stroke
@@
 	(wire
 		(pts
+			(xy 377.19 177.8) (xy 386.08 177.8)
+		)
+		(stroke
+			(width 0)
+			(type default)
+		)
+	)
+	(wire
+		(pts
 			(xy 107.95 201.93) (xy 92.71 201.93)
 		)
@@
 	(wire
 		(pts
+			(xy 377.19 167.64) (xy 386.08 167.64)
+		)
+		(stroke
+			(width 0)
+			(type default)
+		)
+	)
+	(wire
+		(pts
 			(xy 59.69 220.98) (xy 139.7 220.98)
 		)
@@
 	(wire
 		(pts
+			(xy 377.19 177.8) (xy 377.19 179.07)
+		)
+		(stroke
+			(width 0)
+			(type default)
+		)
+	)
+	(wire
+		(pts
 			(xy 68.58 39.37) (xy 68.58 43.18)
 		)
@@
 					(unit 1)
 				)
+			)
+		)
+	)
+	(symbol
+		(lib_id "Simulation_SPICE:VSIN")
+		(at 386.08 172.72 0)
+		(unit 1)
+		(exclude_from_sim no)
+		(in_bom yes)
+		(on_board yes)
+		(dnp no)
+		(fields_autoplaced yes)
+		(property "Reference" "V1"
+			(at 389.89 170.0501 0)
+			(effects
+				(font
+					(size 1.27 1.27)
+				)
+				(justify left)
+			)
+		)
+		(property "Value" "VSIN"
+			(at 389.89 172.5901 0)
+			(effects
+				(font
+					(size 1.27 1.27)
+				)
+				(justify left)
+			)
+		)
+		(property "Footprint" ""
+			(at 386.08 172.72 0)
+			(effects
+				(font
+					(size 1.27 1.27)
+				)
+				(hide yes)
+			)
+		)
+		(property "Datasheet" "https://ngspice.sourceforge.io/docs/ngspice-html-manual/manual.xhtml#sec_Independent_Sources_for"
+			(at 386.08 172.72 0)
+			(effects
+				(font
+					(size 1.27 1.27)
+				)
+				(hide yes)
+			)
+		)
+		(property "Description" "Voltage source, sinusoidal"
+			(at 386.08 172.72 0)
+			(effects
+				(font
+					(size 1.27 1.27)
+				)
+				(hide yes)
+			)
+		)
+		(property "Sim.Pins" "1=+ 2=-"
+			(at 386.08 172.72 0)
+			(effects
+				(font
+					(size 1.27 1.27)
+				)
+				(hide yes)
+			)
+		)
+		(property "Sim.Params" "dc=0 ampl=311 f=50 ac=1"
+			(at 389.89 175.1301 0)
+			(effects
+				(font
+					(size 1.27 1.27)
+				)
+				(justify left)
+			)
+		)
+		(property "Sim.Type" "SIN"
+			(at 386.08 172.72 0)
+			(effects
+				(font
+					(size 1.27 1.27)
+				)
+				(hide yes)
+			)
+		)
+		(property "Sim.Device" "V"
+			(at 386.08 172.72 0)
+			(effects
+				(font
+					(size 1.27 1.27)
+				)
+				(justify left)
+				(hide yes)
+			)
+		)
+		(pin "1"
+		)
+		(pin "2"
+		)
+		(instances
+			(project ""
+				(path "/ea3996f2-7d6b-4a86-86ab-4ed62213f41f"
+					(reference "V1")
+					(unit 1)
+				)
