File: KiCad/3dFilamentDryer/3dFilamentDryer.kicad_sch (KiCad schematic)
At the start: 53 parts, among them J1 ILI9341 Connection Port, J2 FTDI, J3 Mains, J4 Fan, J5 MAX6675, K1 SRD-05VDC-SL-C, Q1 BTA12-600BW, Q2 S8050-J3Y, Q3 S8050-J3Y, Q4 BC817-25-HT, U1 4N28, U2 TLV1117-33, U3 ESP32-WROOM-32E-N4, U5 MOC3053M, U6 SN74LVC1G14DBVR

Commit message: PCB fix
Connections:
- net FAN: now also U3.16 (IO13); no longer U3.14 (IO12)
- net VSPI_SCK: now reaches J1.10 (T_CLK), J1.7 (SCK), J5.3 (Pin_3)
- net VSPI_SCK: now also U3.30 (IO18); no longer U3.20 (SCK/CLK)
- net SENSOR_CS: now reaches J5.4 (Pin_4)
- net SENSOR_CS: now also U3.11 (IO26); no longer U3.16 (IO13)
- net VSPI_MISO: now reaches J1.13 (T_DO), J1.9 (SDO(MISO)), J5.5 (Pin_5)
- net VSPI_MISO: now also U3.31 (IO19); no longer U3.22 (SDI/SD1)
- net VSPI_MOSI: now reaches J1.12 (T_DIN), J1.6 (SDI(MOSI))
- net VSPI_MOSI: now also U3.37 (IO23); no longer U3.21 (SDO/SD0)
- net at J1.3 (CS): now also U3.26 (IO4); no longer U3.23 (IO15)
- net at J1.4 (RESET): now also U3.13 (IO14); no longer U3.26 (IO4)
- net at J1.5 (DC): now also U3.27 (IO16); no longer U3.24 (IO2)
Other:
- moved on the sheet: J3, J5, V1

Commit message: Signed-off-by: omerkaraoglu <omerdjns@gmail.com>
Other:
- company: Elektromag Makine -> READARK
Changed lines of the file:
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@@
 	(title_block
 		(title "3D Printer Filament Dryer & Print Annealer")
-		(date "2026-03-04")
-		(rev "1.2")
-		(company "Elektromag Makine")
+		(date "2026-04-13")
+		(rev "1.3")
+		(company "READARK")
 		(comment 1 "M. Ömer Karaoğlu")
 	)

Commit message: Firmware v2.1.2 Hardware Rev2
Parts:
- removed F2: 250VAC 1A Slow Blow, Fuse:Fuseholder_Clip-5x20mm_Littelfuse_445-030_Inline_P20.50x5.20mm_D1.30mm_Horizontal, symbol Device:Fuse
- removed F4: 250VAC 2.5A Normal, Fuse:Fuseholder_Clip-5x20mm_Littelfuse_445-030_Inline_P20.50x5.20mm_D1.30mm_Horizontal, symbol Device:Fuse
- F3: value 250VAC 2.5A Normal -> 250VAC 8A Normal
- R1: value Heater 500W -> Heater 1300W
Connections:
- net NEUT: now also C1.2, L1.1, R1.2, RV1.2
Other:
- moved on the sheet: R1
